File: breadboard_power_supply.kicad_pcb (KiCad board)
At the start: 2 copper layers, 31.1 x 52.5 mm, 17 parts, among them J1 Conn_01x02_Pin, J2 Conn_01x02_Pin, J3 Conn_01x03_Pin, J4 Conn_01x03_Pin, J5 Screw_Terminal_01x02, J6 Barrel_Jack_Switch, J7 Screw_Terminal_01x02, U2 LM317_TO-220, U3 LM7805_TO220

Commit message: v0.1
Connections:
- J1 pad 2: /PWR_OUT -> /PWR_OUT_BOT
- J2 pad 2: /PWR_OUT -> /PWR_OUT_TOP
- J3 pad 2: /PWR_OUT -> /PWR_OUT_BOT
- J4 pad 2: /PWR_OUT -> /PWR_OUT_TOP
- J5 pad 2: /PWR_OUT -> /PWR_OUT_BOT
- J7 pad 2: /PWR_OUT -> /PWR_OUT_TOP
Routing:
- net /PWR_OUT: track 99.0 -> 0.00 mm
- net /PWR_OUT_BOT: track 0.00 -> 27.2 mm
- net /PWR_OUT_TOP: track 0.00 -> 26.1 mm
Other:
- board text added: "3.3v"
- board text added: "5v"
Changed lines of the file:
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@@
 			(outputformat 1)
 			(mirror no)
-			(drillshape 1)
+			(drillshape 0)
 			(scaleselection 1)
-			(outputdirectory "")
+			(outputdirectory "gerbers/")
 		)
 	)
@@
 	(net 4 "/3v3")
 	(net 5 "Net-(D1-A)")
-	(net 6 "/PWR_OUT")
+	(net 6 "/PWR_OUT_TOP")
 	(net 7 "/PWR_IN")
 	(net 8 "Net-(U2-ADJ)")
 	(net 9 "unconnected-(S1-Pad3)")
+	(net 10 "/PWR_OUT_BOT")
 	(footprint "Package_TO_SOT_THT:TO-220-3_Vertical"
 		(layer "F.Cu")
@@
 		(property "Value" "LM7805_TO220"
 			(at 2.54 2.5 0)
-			(layer "F.Fab")
+			(layer "F.SilkS")
 			(effects
 				(font
@@
 		)
 		(property ki_fp_filters "TO?220*")
-		(sheetname "Root")
+		(sheetname "Raiz")
 		(sheetfile "breadboard_power_supply.kicad_sch")
 		(attr through_hole)
@@
 			)
 		)
-		(sheetname "Root")
+		(sheetname "Raiz")
 		(sheetfile "breadboard_power_supply.kicad_sch")
 		(attr through_hole)
@@
 		)
 		(property ki_fp_filters "TerminalBlock*:*")
-		(sheetname "Root")
+		(sheetname "Raiz")
 		(sheetfile "breadboard_power_supply.kicad_sch")
 		(attr through_hole)
@@
 			(layers "*.Cu" "*.Mask")
 			(remove_unused_layers no)
-			(net 6 "/PWR_OUT")
+			(net 10 "/PWR_OUT_BOT")
 			(pinfunction "Pin_2")
 			(pintype "passive")
@@
 		(tags "C Disc series Radial pin pitch 2.50mm  diameter 3.0mm width 1.6mm Capacitor")
 		(property "Reference" "C3"
-			(at 1.25 -2.05 180)
+			(at 2.8536 -1.9738 180)
 			(layer "F.SilkS")
 			(effects
@@
 		)
 		(property "Value" "1u"
-			(at 1.25 2.05 180)
-			(layer "F.Fab")
+			(at 0.5286 -1.9488 180)
+			(layer "F.SilkS")
 			(effects
 				(font
@@
 		)
 		(property ki_fp_filters "C_*")
-		(sheetname "Root")
+		(sheetname "Raiz")
 		(sheetfile "breadboard_power_supply.kicad_sch")
 		(attr through_hole)
@@
 			(at -2.6974 2.4742 0)
 			(layer "F.SilkS")
+			(hide yes)
 			(effects
 				(font
@@
 			)
 		)
-		(property "Purpose" "Output Voltage Selector 2"
+		(property "Purpose" "Output Voltage Selector 1"
 			(at 0 0 90)
 			(unlocked yes)
@@
 		)
 		(property ki_fp_filters "Connector*:*_1x??_*")
-		(sheetname "Root")
+		(sheetname "Raiz")
 		(sheetfile "breadboard_power_supply.kicad_sch")
 		(attr through_hole)
@@
 			(layers "*.Cu" "*.Mask")
 			(remove_unused_layers no)
-			(net 6 "/PWR_OUT")
+			(net 6 "/PWR_OUT_TOP")
 			(pinfunction "Pin_2")
 			(pintype "passive")
@@
 		)
 		(property ki_fp_filters "TerminalBlock*:*")
-		(sheetname "Root")
+		(sheetname "Raiz")
 		(sheetfile "breadboard_power_supply.kicad_sch")
 		(attr through_hole)
@@
 			(layers "*.Cu" "*.Mask")
 			(remove_unused_layers no)
-			(net 6 "/PWR_OUT")
+			(net 6 "/PWR_OUT_TOP")
 			(pinfunction "Pin_2")
 			(pintype "passive")
@@
 		(tags "Through hole pin header THT 1x02 2.54mm single row")
 		(property "Reference" "J1"
-			(at -2.9972 0.9652 0)
+			(at -3.261 1.1832 0)
 			(layer "F.SilkS")
 			(effects
@@
 		)
 		(property ki_fp_filters "Connector*:*_1x??_*")
-		(sheetname "Root")
+		(sheetname "Raiz")
 		(sheetfile "breadboard_power_supply.kicad_sch")
 		(attr through_hole)
@@
 			(layers "*.Cu" "*.Mask")
 			(remove_unused_layers no)
-			(net 6 "/PWR_OUT")
+			(net 10 "/PWR_OUT_BOT")
 			(pinfunction "Pin_2")
 			(pintype "passive")
@@
 		(property "Value" "LM317_TO-220"
 			(at 2.54 2.5 180)
-			(layer "F.Fab")
+			(layer "F.SilkS")
 			(effects
 				(font
@@
 		)
 		(property ki_fp_filters "TO?220*")
-		(sheetname "Root")
+		(sheetname "Raiz")
 		(sheetfile "breadboard_power_supply.kicad_sch")
 		(attr through_hole)
@@
 		(tags "C Disc series Radial pin pitch 2.50mm  diameter 3.0mm width 1.6mm Capacitor")
 		(property "Reference" "C2"
-			(at 1.3208 2.032 180)
+			(at 2.906 2.0084 180)
 			(layer "F.SilkS")
 			(effects
@@
 		)
 		(property "Value" "0.1u"
-			(at 1.25 2.05 180)
-			(layer "F.Fab")
+			(at -0.244 1.9334 180)
+			(layer "F.SilkS")
 			(effects
 				(font
@@
 		)
 		(property ki_fp_filters "C_*")
-		(sheetname "Root")
+		(sheetname "Raiz")
 		(sheetfile "breadboard_power_supply.kicad_sch")
 		(attr through_hole)
@@
 			(at 2.3976 2.9392 0)
 			(layer "F.SilkS")
+			(hide yes)
 			(effects
 				(font
@@
 		)
 		(property ki_fp_filters "Connector*:*_1x??_*")
-		(sheetname "Root")
+		(sheetname "Raiz")
 		(sheetfile "breadboard_power_supply.kicad_sch")
 		(attr through_hole)
@@
 			(layers "*.Cu" "*.Mask")
 			(remove_unused_layers no)
-			(net 6 "/PWR_OUT")
+			(net 10 "/PWR_OUT_BOT")
 			(pinfunction "Pin_2")
 			(pintype "passive")
@@
 		)
 		(property ki_fp_filters "BarrelJack*")
-		(sheetname "Root")
+		(sheetname "Raiz")
 		(sheetfile "breadboard_power_supply.kicad_sch")
 		(attr through_hole)
@@
 		)
 		(property ki_fp_filters "Connector*:*_1x??_*")
-		(sheetname "Root")
+		(sheetname "Raiz")
 		(sheetfile "breadboard_power_supply.kicad_sch")
 		(attr through_hole)
@@
 			(layers "*.Cu" "*.Mask")
 			(remove_unused_layers no)
-			(net 6 "/PWR_OUT")
+			(net 6 "/PWR_OUT_TOP")
 			(pinfunction "Pin_2")
 			(pintype "passive")
@@
 		(tags "Resistor Axial_DIN0204 series Axial Horizontal pin pitch 7.62mm 0.167W length 3.6mm diameter 1.6mm")
 		(property "Reference" "R3"
-			(at 9.3356 0 0)
+			(at 3.79 0.0614 90)
 			(layer "F.SilkS")
 			(effects
@@
 		)
 		(property "Value" "560"
-			(at 3.81 1.92 -90)
-			(layer "F.Fab")
+			(at 10.215 0.0614 270)
+			(layer "F.SilkS")
 			(effects
 				(font
@@
 		)
 		(property ki_fp_filters "R_*")
-		(sheetname "Root")
+		(sheetname "Raiz")
 		(sheetfile "breadboard_power_supply.kicad_sch")
 		(attr through_hole)
@@
 		(tags "Resistor Axial_DIN0204 series Axial Horizontal pin pitch 7.62mm 0.167W length 3.6mm diameter 1.6mm")
 		(property "Reference" "R1"
-			(at 3.81 -1.92 90)
+			(at 3.81 -0.041 90)
 			(layer "F.SilkS")
 			(effects
@@
 		)
 		(property "Value" "330"
-			(at 3.81 1.92 90)
-			(layer "F.Fab")
+			(at 3.788 -1.816 90)
+			(layer "F.SilkS")
 			(effects
 				(font
@@
 		)
 		(property ki_fp_filters "R_*")
-		(sheetname "Root")
+		(sheetname "Raiz")
 		(sheetfile "breadboard_power_supply.kicad_sch")
 		(attr through_hole)
@@
 		)
 		(property ki_fp_filters "LED* LED_SMD:* LED_THT:*")
-		(sheetname "Root")
+		(sheetname "Raiz")
 		(sheetfile "breadboard_power_supply.kicad_sch")
 		(attr through_hole)
@@
 		(tags "Resistor Axial_DIN0204 series Axial Horizontal pin pitch 7.62mm 0.167W length 3.6mm diameter 1.6mm")
 		(property "Reference" "R2"
-			(at 9.3356 -0.0508 0)
+			(at 3.74 0.0562 90)
 			(layer "F.SilkS")
 			(effects
@@
 		)
 		(property "Value" "330"
-			(at 3.81 1.92 -90)
-			(layer "F.Fab")
+			(at 10.24 0.1312 270)
+			(layer "F.SilkS")
 			(effects
 				(font
@@
 		)
 		(property ki_fp_filters "R_*")
-		(sheetname "Root")
+		(sheetname "Raiz")
 		(sheetfile "breadboard_power_supply.kicad_sch")
 		(attr through_hole)
@@
 		(tags "C Disc series Radial pin pitch 2.50mm  diameter 3.0mm width 1.6mm Capacitor")
 		(property "Reference" "C1"
-			(at 1.25 -2.05 0)
+			(at 0.0816 -1.9834 0)
 			(layer "F.SilkS")
 			(effects
@@
 		)
 		(property "Value" "10u"
-			(at 1.25 2.05 0)
-			(layer "F.Fab")
+			(at 2.6316 -2.0084 0)
+			(layer "F.SilkS")
 			(effects
 				(font
@@
 		)
 		(property ki_fp_filters "C_*")
-		(sheetname "Root")
+		(sheetname "Raiz")
 		(sheetfile "breadboard_power_supply.kicad_sch")
 		(attr through_hole)
@@
 		(layer "Edge.Cuts")
 	)
+	(gr_text "5v"
+		(at 107.35 128.7587 0)
+		(layer "F.SilkS")
+		(effects
+			(font
+				(size 1 1)
+				(thickness 0.1)
+			)
+			(justify left bottom)
+		)
+	)
+	(gr_text "3.3v"
+		(at 100.9 128.7587 0)
+		(layer "F.SilkS")
+		(effects
+			(font
+				(size 1 1)
+				(thickness 0.1)
+			)
+			(justify left bottom)
+		)
+	)
+	(gr_text "3.3v"
+		(at 100.75 85.5279 0)
+		(layer "F.SilkS")
+		(effects
+			(font
+				(size 1 1)
+				(thickness 0.1)
+			)
+			(justify left bottom)
+		)
+	)
+	(gr_text "5v"
+		(at 107.2 85.5279 0)
+		(layer "F.SilkS")
+		(effects
+			(font
+				(size 1 1)
+				(thickness 0.1)
+			)
+			(justify left bottom)
+		)
+	)
 	(segment
 		(start 119.634 109.982)
@@
 	)
 	(segment
-		(start 122.586 130.6068)
-		(end 129.286 130.6068)
-		(width 0.2)
-		(layer "F.Cu")
-		(net 6)
-	)
-	(segment
 		(start 117.046 81.141)
 		(end 120.396 84.491)
@@
 	)
 	(segment
-		(start 117.046 131.7668)
-		(end 105.9576 131.7668)
-		(width 0.2)
-		(layer "F.Cu")
-		(net 6)
-	)
-	(segment
-		(start 120.396 128.4168)
-		(end 122.5136 126.2992)
-		(width 0.2)
-		(layer "F.Cu")
-		(net 6)
-	)
-	(segment
 		(start 106.3718 81.141)
 		(end 117.046 81.141)
@@
 	)
 	(segment
-		(start 122.5136 86.6086)
-		(end 120.396 84.491)
-		(width 0.2)
-		(layer "F.Cu")
-		(net 6)
-	)
-	(segment
-		(start 105.9576 131.7668)
-		(end 104.8076 130.6168)
-		(width 0.2)
-		(layer "F.Cu")
-		(net 6)
-	)
-	(segment
-		(start 122.5136 126.2992)
-		(end 122.5136 86.6086)
-		(width 0.2)
-		(layer "F.Cu")
-		(net 6)
-	)
-	(segment
-		(start 120.396 128.4168)
-		(end 122.586 130.6068)
-		(width 0.2)
-		(layer "F.Cu")
-		(net 6)
-	)
-	(segment
-		(start 120.396 128.4168)
-		(end 117.046 131.7668)
-		(width 0.2)
-		(layer "F.Cu")
-		(net 6)
-	)
-	(segment
 		(start 129.286 84.831)
 		(end 120.736 84.831)
@@
 		(net 8)
 	)
+	(segment
+		(start 122.586 130.6068)
+		(end 129.286 130.6068)
+		(width 0.2)
+		(layer "F.Cu")
+		(net 10)
+	)
+	(segment
+		(start 117.046 131.7668)
+		(end 105.9576 131.7668)
+		(width 0.2)
+		(layer "F.Cu")
+		(net 10)
+	)
+	(segment
+		(start 105.9576 131.7668)
+		(end 104.8076 130.6168)
+		(width 0.2)
+		(layer "F.Cu")
+		(net 10)
+	)
+	(segment
+		(start 120.396 128.4168)
+		(end 122.586 130.6068)
+		(width 0.2)
+		(layer "F.Cu")
+		(net 10)
+	)
+	(segment
+		(start 120.396 128.4168)
+		(end 117.046 131.7668)
+		(width 0.2)
+		(layer "F.Cu")
+		(net 10)
+	)
 	(zone
